File: hw/motor_node.sch (EAGLE design)
At the start: 51 parts, among them IC1 TINY84 or TINY841, IC3 MCP1703DB, Q1 BSS138, Q2 BSS138, Q3 BSS138

Commit message: -
Parts:
- added 100K, 10K: 10k, rcl:R-EU_M0805
- added C6: 100n, rcl:C-EUC0805
- added P_UM: (no value), wirepad:1,6/0,8
Connections:
- new net N$2: 100K.1, P_UM.P
- net GND: now also 10K.1, C6.1
- net PA0: now also 100K.2, 10K.2, C6.2
Changed lines of the file:
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@@
 <?xml version="1.0" encoding="utf-8"?>
 <!DOCTYPE eagle SYSTEM "eagle.dtd">
-<eagle version="9.5.2">
+<eagle version="9.6.2">
 <drawing>
 <settings>
@@
 <setting verticaltext="up"/>
 </settings>
-<grid distance="0.1" unitdist="inch" unit="mil" style="lines" multiple="1" display="no" altdistance="50" altunitdist="mil" altunit="mil"/>
+<grid distance="50" unitdist="mil" unit="mil" style="lines" multiple="1" display="no" altdistance="0.01" altunitdist="inch" altunit="inch"/>
 <layers>
 <layer number="1" name="Top" color="4" fill="1" visible="no" active="no"/>
@@
 <part name="J_PB2B" library="SparkFun-Jumpers" deviceset="JUMPER-SMT_2_NO" device="_NO-SILK" package3d_urn="urn:adsk.eagle:package:39277/1" value=""/>
 <part name="D2" library="diode" library_urn="urn:adsk.eagle:library:210" deviceset="DIODE-" device="MINIMELF" package3d_urn="urn:adsk.eagle:package:43429/2"/>
+<part name="100K" library="rcl" library_urn="urn:adsk.eagle:library:334" deviceset="R-EU_" device="M0805" package3d_urn="urn:adsk.eagle:package:23556/2" value="10k"/>
+<part name="10K" library="rcl" library_urn="urn:adsk.eagle:library:334" deviceset="R-EU_" device="M0805" package3d_urn="urn:adsk.eagle:package:23556/2" value="10k"/>
+<part name="C6" library="rcl" deviceset="C-EU" device="C0805" value="100n"/>
+<part name="GND19" library="supply1" deviceset="GND" device=""/>
+<part name="GND20" library="supply1" deviceset="GND" device=""/>
+<part name="P_UM" library="wirepad" library_urn="urn:adsk.eagle:library:412" deviceset="1,6/0,8" device="" package3d_urn="urn:adsk.eagle:package:30830/1"/>
 </parts>
 <sheets>
@@
 <attribute name="VALUE" x="83.82" y="99.2886" size="1.778" layer="96"/>
 </instance>
+<instance part="100K" gate="G$1" x="82.55" y="162.56" smashed="yes">
+<attribute name="NAME" x="78.74" y="164.0586" size="1.778" layer="95"/>
+<attribute name="VALUE" x="78.74" y="159.258" size="1.778" layer="96"/>
+</instance>
+<instance part="10K" gate="G$1" x="87.63" y="157.48" smashed="yes" rot="R90">
+<attribute name="NAME" x="86.1314" y="153.67" size="1.778" layer="95" rot="R90"/>
+<attribute name="VALUE" x="90.932" y="153.67" size="1.778" layer="96" rot="R90"/>
+</instance>
+<instance part="C6" gate="G$1" x="96.52" y="154.94" smashed="yes" rot="R180">
+<attribute name="NAME" x="94.996" y="154.559" size="1.778" layer="95" rot="R180"/>
+<attribute name="VALUE" x="94.996" y="159.639" size="1.778" layer="96" rot="R180"/>
+</instance>
+<instance part="GND19" gate="1" x="87.63" y="149.86" smashed="yes">
+<attribute name="VALUE" x="85.09" y="147.32" size="1.778" layer="96"/>
+</instance>
+<instance part="GND20" gate="1" x="96.52" y="149.86" smashed="yes">
+<attribute name="VALUE" x="93.98" y="147.32" size="1.778" layer="96"/>
+</instance>
+<instance part="P_UM" gate="P" x="72.39" y="162.56" smashed="yes">
+<attribute name="NAME" x="71.247" y="164.4142" size="1.778" layer="95"/>
+<attribute name="VALUE" x="71.247" y="159.258" size="1.778" layer="96"/>
+</instance>
 </instances>
 <busses>
@@
 <pinref part="IC2" gate="G$1" pin="GND"/>
 <pinref part="GND13" gate="1" pin="GND"/>
+</segment>
+<segment>
+<pinref part="10K" gate="G$1" pin="1"/>
+<pinref part="GND19" gate="1" pin="GND"/>
+</segment>
+<segment>
+<pinref part="GND20" gate="1" pin="GND"/>
+<pinref part="C6" gate="G$1" pin="1"/>
 </segment>
 </net>
@@
 <junction x="78.74" y="71.12"/>
 </segment>
+<segment>
+<pinref part="100K" gate="G$1" pin="2"/>
+<pinref part="10K" gate="G$1" pin="2"/>
+<pinref part="C6" gate="G$1" pin="2"/>
+<wire x1="87.63" y1="162.56" x2="96.52" y2="162.56" width="0.1524" layer="91"/>
+<wire x1="96.52" y1="162.56" x2="96.52" y2="160.02" width="0.1524" layer="91"/>
+<junction x="87.63" y="162.56"/>
+<label x="96.52" y="162.56" size="1.778" layer="95" xref="yes"/>
+</segment>
 </net>
 <net name="PA1" class="0">
@@
 </segment>
 </net>
+<net name="N$2" class="0">
+<segment>
+<pinref part="100K" gate="G$1" pin="1"/>
+<pinref part="P_UM" gate="P" pin="P"/>
+<wire x1="74.93" y1="162.56" x2="77.47" y2="162.56" width="0.1524" layer="91"/>
+</segment>
+</net>
