File: hw/uni_node.sch (EAGLE design)
At the start: 4 parts, among them U1 TINY45, X1 BUS

Commit message: -
Parts:
- removed C1: 100n, rcl:C-EUC0805
- removed SV1: (no value), con-lstb:MA06-1
- removed U1: TINY45, avr-7:TINY25/45/85-20SU
- added C2: 100n, rcl:C-EUC0805
- added CS, DW, GND, GND_, INT, INT0, PA0, PA1, PA2, PA3, PA7, PAD1, PAD10, PAD100, PAD101, PAD102, PAD11, PAD12, PAD13, PAD14, PAD15, PAD16, PAD17, PAD18, PAD19, PAD2, PAD20, PAD21, PAD22, PAD23, PAD24, PAD25, PAD26, PAD27, PAD28, PAD29, PAD3, PAD30, PAD31, PAD32, PAD33, PAD34, PAD35, PAD36, PAD37, PAD38, PAD39, PAD4, PAD40, PAD41, PAD42, PAD43, PAD44, PAD45, PAD46, PAD47, PAD48, PAD49, PAD5, PAD50, PAD51, PAD52, PAD53, PAD54, PAD55, PAD56, PAD57, PAD58, PAD59, PAD6, PAD60, PAD61, PAD62, PAD63, PAD64, PAD65, PAD66, PAD67, PAD68, PAD69, PAD7, PAD70, PAD71, PAD72, PAD73, PAD74, PAD75, PAD76, PAD77, PAD78, PAD79, PAD8, PAD80, PAD81, PAD82, PAD83, PAD84, PAD85, PAD86, PAD87, PAD88, PAD89, PAD9, PAD90, PAD91, PAD92, PAD93, PAD94, PAD95, PAD96, PAD97, PAD98, PAD99, PB0, PB1, SCL, SDA, VCC: (no value), wirepad:1,6/0,9
- added D2: (no value), diode:DIODE-MINIMELF
- added IC1: TINY84 or TINY841, avr-7:TINY24/44/84-SSU
- added J_CS: JUMPER-SMT_3_1-NC_PASTE_NO-SILK, SparkFun-Jumpers:JUMPER-SMT_3_1-NC_PASTE_NO-SILK
- added R1, R2, R3, R4, R5: 10k, rcl:R-EU_M0805
Connections:
- removed net INT_MISO: U1.(OCP)PB1, X1-1.S
- removed net PB3: SV1.6, U1.(ADC3)PB3
- removed net PB4: SV1.1, U1.(ADC2)PB4
- removed net RESET: U1.(ADC0)PB5, X1-5.S
- removed net SCL_SCK: SV1.3, U1.(ADC1)PB2, X1-3.S
- removed net SDA_MOSI: SV1.2, U1.(AREF)PB0, X1-4.S
- new net BUS_INT: IC1.(PCINT5/OC1B/MISO/DO/ADC5)PA5, INT.P, R4.2, X1-1.S
- new net BUS_P5: CS.P, J_CS.2, R5.2, X1-5.S
- new net BUS_RESET: D2.C, J_CS.3
- new net BUS_SCL: IC1.(PCINT4/T1/SCL/USCK/ADC4)PA4, R3.2, SCL.P, X1-3.S
- new net BUS_SDA: IC1.(PCINT6/OC1A/SDA/MOSI/ADC6)PA6, R2.2, SDA.P, X1-4.S
- new net DW: D2.A, DW.P, IC1.(PCINT11/RESET/DW)PB3, R1.2
- new net INT0: IC1.(PCINT10/INT0/OC0A/CKOUT)PB2, INT0.P, J_CS.1
- new net PA0: IC1.(PCINT0/AREF/ADC0)PA0, PA0.P
- new net PA1: IC1.(PCINT1/AIN0/ADC1)PA1, PA1.P
- new net PA2: IC1.(PCINT2/AIN1/ADC2)PA2, PA2.P
- new net PA3: IC1.(PCINT3/T0/ADC3)PA3, PA3.P
- new net PA7: IC1.(PCINT7/ICP/OC0B/ADC7)PA7, PA7.P
- new net PB0: IC1.(PCINT8/XTAL1/CLKI)PB0, PB0.P
- new net PB1: IC1.(PCINT9/XTAL2)PB1, PB1.P
- net GND: now also C2.2, GND.P, GND_.P, IC1.GND, PAD100.P, PAD101.P, PAD102.P; no longer C1.2, SV1.5, U1.GND
- net VCC: now also C2.1, IC1.VCC, R1.1, R2.1, R3.1, R4.1, R5.1, VCC.P; no longer C1.1, SV1.4, U1.VCC
Other:
- note added: "V1.0"
