File: hw/main_node.sch (EAGLE design)
At the start: 21 parts, among them IC10 ESP32-WROVER

Commit message: some files updated
Parts:
- added C10: 100uF/6V, rcl:CPOL-EUB/3528-21R
- added C11, C3, C8: 0.1, rcl:C-EUC0805
- added D1: 4148, diode:DIODE-MINIMELF
- added D2, D3, D4, D5, D6, D7: (no value), diode:DIODE-MELF-MLL41
- added F1: FUSE 6A, fuse:FUSESH22,5A
- added IC2: (no value), arduino:ARDUINO2009_22
- added IC3: MEGA48/88/168-AU, avr-6:MEGA48/88/168-AU
- added IC5: STM32G081RBT6, stm32:STM32G081RBT6
- added J_L1, J_L2, J_L3, J_L4, J_L5, J_L6, J_L7, J_L7B, J_L8, J_L8B, J_R6, J_R7, J_R8, J_VCCOUT, SJ12: (no value), jumper:SJ
- added J_VCC, SJ13: (no value), jumper:SJ2W
- added L, R: (no value), con-lstb:MA08-1
- added LED1A, LED1B: (no value), led:LED5MM
- added LED2: (no value), led:LEDCHIPLED_0805
- added Q1, Q2: IRF9530, transistor-fet:IRF9530
- added Q4: (no value), crystal:CRYSTALTC26V
- added R10, R19, R32, R33, R34, R35, R36, R37: (no value), rcl:R-EU_R0805
- added R11: (no value), rcl:R-EU_R0603
- added R18: 470, rcl:R-EU_R0805
- added R2, R9: 10k, rcl:R-EU_R0805
- added R23: 68, rcl:R-EU_R0805
- added R3, R4, R5, R6, R7, R8: (no value), rcl:R-EU_R2512
- added T2: (no value), transistor:BC817-16-NPN-SOT23-BEC
- added X1: (no value), con-wago-508:W237-08P
- IC1: value (none) -> MCP1703DB; device arduino:ARDUINO2009_PIN_21 -> linear:MCP1703DB
Connections:
- new net ADC0: IC5G$1.PA0
- new net ADC1: IC5G$1.PA1
- new net BNO055_RESET: IC5G$7.PD2
- new net BUS_FON: IC5G$4.PB14
- new net BUS_INT: J_R8.2
- new net BUS_RESET: IC5G$7.PD1, J_L8.1
- new net BUS_SCL: J_R7.2
- new net BUS_SDA: J_R6.2
- new net CHARGE_ON: IC5G$2.PA8
- new net FLASH_CS: IC5G$8.PD9
- new net FLASH_HOLD: IC5G$7.PD5
- new net FLASH_WP: IC5G$7.PD6
- new net INT: IC5G$6.PC15
- new net LED1: IC5G$5.PC1, LED1B.A
- new net LED2: IC5G$1.PA2, R11.2
- new net LEDSTRB: R18.1
- new net LIDAR_M: IC5G$7.PD0
- new net LIDAR_RX: IC5G$1.PA3
- new net L_RST_0: IC5G$7.PD3
- new net L_RST_1: IC5G$3.PB1
- new net L_RST_10: IC5G$1.PA4, IC5G$4.PB12
- new net L_RST_11: IC5G$4.PB13
- new net L_RST_2: IC5G$7.PD4
- new net L_RST_3: IC5G$3.PB3
- new net L_RST_4: IC5G$3.PB4
- new net L_RST_5: IC5G$3.PB5
- new net L_RST_6: IC5G$3.PB6
- new net L_RST_7: IC5G$3.PB7
- new net L_RST_8: IC5G$5.PC7
- new net L_RST_9: IC5G$5.PC6
- new net N$1: Q1.G, Q2.G, R10.2, T2.C
- new net N$10: IC2G$1.A2
- new net N$11: IC2G$1.A3
- new net N$12: J_R8.1, R.8
- new net N$13: IC2G$1.A4
- new net N$14: IC2G$1.A5
- new net N$15: IC2G$1.0
- new net N$16: IC2G$1.1
- new net N$17: IC2G$1.2
- new net N$18: IC2G$1.3
- new net N$19: IC2G$1.4
- new net N$2: IC3.PC5(ADC5/SCL/PCINT13)
- new net N$20: IC2G$1.5
- new net N$21: IC2G$1.6
- new net N$22: IC2G$1.7
- new net N$23: IC2G$1.8
- new net N$24: J_L7.2, J_L7B.2, L.7
- new net N$25: J_L6.2, L.6, R19.1
- new net N$26: IC2G$1.9
- new net N$27: J_L8.2, J_L8B.2, L.8
- new net N$28: J_L5.2, L.5, R34.1
- new net N$29: J_L4.2, L.4, R35.1
- new net N$3: IC3.PC4(ADC4/SDA/PCINT12)
- new net N$30: J_L2.2, L.2, R37.1
- new net N$31: J_L3.2, L.3, R36.1
- new net N$32: J_L1.2, L.1
- new net N$33: IC2G$1.10
- new net N$34: IC2G$1.11
- new net N$35: IC2G$1.12
- new net N$36: IC2G$1.13
- new net N$37: IC2G$1.AREF
- new net N$38: IC2G$1.!RESET
- new net N$39: IC5G$9.OSC_IN, Q4.1, SJ12.2
- new net N$4: IC3.PB2(SS/OC1B/PCINT2)
- new net N$40: IC5G$9.VDDA, IC5G$9.VREF+, SJ13.2
- new net N$41: IC5G$8.PD8, R18.2
- new net N$42: LED1A.A, LED1B.C
- new net N$43: LED1A.C, R23.1
- new net N$44: IC5G$9.OSC_OUT, Q4.2
- new net N$45: LED2.A, R11.1
- new net N$46: IC3.PB5(SCK/PCINT5)
- new net N$47: IC3.PB4(MISO/PCINT4)
- new net N$48: IC3.PB3(MOSI/OC2A/PCINT3)
- new net N$49: IC3.PD1(TXD/PCINT17)
- new net N$5: J_R6.1, R.6
- new net N$50: IC3.PD0(RXD/PCINT16)
- new net N$51: R2.2, R9.1, T2.B
- new net N$52: IC3.PD2(INT0/PCINT18)
- new net N$6: J_R7.1, R.7
- new net N$8: IC2G$1.A0
- new net N$9: IC2G$1.A1
- new net OLED_SCL: J_L8B.1
- new net OLED_SDA: J_L7B.1
- new net PON1: R2.1
- new net SCL: IC5G$2.PA9
- new net SDA: IC5G$2.PA10
- new net SPI2_MISO: IC5G$5.PC2
- new net SPI2_MOSI: IC5G$5.PC3
- new net SPI2_NSS: IC5G$4.PB9
- new net SPI2_SCK: IC5G$4.PB8
- new net SPI_CS0: J_L5.1
- new net SPI_CS1: J_L6.1
- new net SPI_RESET: J_L7.1
- new net SPI_SCK: J_L4.1
- new net SWCLK: IC5G$2.PA13
- new net SWDIO: IC5G$2.PA14
- new net SWNRES: C11.2, IC5G$9.NRST
- new net U2RXD: R33.2
- new net U2TXD: D1.C
- new net U2_BUS: D1.A, J_L1.1, R32.1, R33.1
- new net U33A: J_VCC.3, J_VCCOUT.2, R.2
- new net U33B: J_VCC.1, R.3
- new net UBAT: F1.1, R.5, X1-7.KL, X1-8.KL
- new net UBATF1: D5.C, F1.2, R5.1, R6.1
- new net UBATF2: C3.1, D2.C, D3.C, D4.C, IC1.VI, Q1.D, Q2.D, R10.1, R5.2, R6.2
- new net UBUS: J_VCCOUT.1
- new net UCH1A: R3.1, X1-4.KL
- new net UCH1B: D2.A, R3.2
- new net UCH2A: R4.1, X1-3.KL
- new net UCH2B: D3.A, R4.2
- new net UOUT1A: D7.C, R7.1, R8.1, X1-5.KL, X1-6.KL
- new net UOUT1B: D6.C, Q1.S, Q2.S, R7.2, R8.2
- new net USTBY: C10.+, C8.1, IC1.VO, IC5G$9.VBAT, SJ13.1
- new net VCC: J_VCC.2, R19.2, R32.2, R34.2, R35.2, R36.2, R37.2
- new net ZUMO_RXD: IC5G$3.PB2
- new net ZUMO_SHDN: IC5G$4.PB15
- new net ZUMO_TXD: IC5G$3.PB0
- net CAM_PWDN: now also IC5G$5.PC0
- net ESP_BOOT: now also SJ12.1
- net ESP_RXD: now also IC5G$5.PC4
- net ESP_TXD: now also IC5G$5.PC5
- net GND: now also C10.-, C11.1, C3.2, C8.2, D4.A, D5.A, D6.A, D7.A, IC1.GND, IC3.AGND, IC3.GND@1, IC3.GND@2, IC5G$9.VSSA, LED2.C, R.1, R23.2, R9.2, T2.E, X1-1.KL, X1-2.KL
- net RPI_11: now also IC5G$6.PC8
- net RPI_12: now also IC5G$6.PC9
- net RPI_13: now also IC5G$6.PC10
- net RPI_14: now also IC5G$6.PC11
- net RPI_15: now also IC5G$6.PC12
- net RPI_16: now also IC5G$6.PC13
- net RPI_18: now also IC5G$6.PC14
- net RPI_CS0: now also IC5G$1.PA6
- net RPI_CS1: now also IC5G$1.PA7
- net SCL2: now also IC5G$4.PB10
- net SDA2: now also IC5G$4.PB11
- net SPI_CLK: now also IC5G$1.PA5
- net SPI_CS: now also IC5G$2.PA15
- net SPI_MISO: now also IC5G$2.PA11, J_L2.1
- net SPI_MOSI: now also IC5G$2.PA12, J_L3.1
- net U3.3: now also SJ13.3
- net U5: now also R.4
