File: hw/motor_node.brd (EAGLE design)
At the start: 27.6 x 27.3 mm, 51 parts, among them IC1 TINY84 or TINY841, IC3 MCP1703DB, Q1 BSS138, Q2 BSS138, Q3 BSS138

Commit message: -
Parts:
- added 100K, 10K: 10k, rcl:M0805
- added C6: 100n, rcl:C0805
- added P_UM: (no value), wirepad:1,6/0,8
Connections:
- new net N$2: 100K.1, P_UM.1
- net GND: now also 10K.1, C6.1
- net PA0: now also 100K.2, 10K.2, C6.2
Routing:
- net PA0: track 8.88 -> 19.8 mm, vias 2 -> 3
- net GND: track 100.0 -> 108.8 mm, vias 21 -> 23
- net VCC: track 69.8 -> 75.7 mm
- net MB_PWM: track 37.9 -> 42.2 mm
- net MB_B: track 24.7 -> 28.8 mm
- net N$2: track 0.00 -> 2.36 mm
- net MA_A: track 36.5 -> 38.5 mm
- net MA_EN__MB_A: track 51.2 -> 52.9 mm
- net SCL_SCK: track 20.7 -> 22.0 mm
- net MA_PWM: track 54.9 -> 55.7 mm

Commit message: some files updated
Changed lines of the file:
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@@
 <setting verticaltext="up"/>
 </settings>
-<grid distance="25" unitdist="mil" unit="mil" style="dots" multiple="1" display="yes" altdistance="1" altunitdist="mil" altunit="mil"/>
+<grid distance="12.5" unitdist="mil" unit="mil" style="dots" multiple="2" display="yes" altdistance="1" altunitdist="mil" altunit="mil"/>
 <layers>
 <layer number="1" name="Top" color="4" fill="1" visible="yes" active="yes"/>
@@
 <wire x1="0" y1="27.295" x2="0" y2="0" width="0" layer="20"/>
 <text x="6.35" y="0.635" size="0.4064" layer="25">Motor Node V1.0</text>
+<wire x1="0" y1="0" x2="27.6225" y2="0" width="0.1524" layer="20"/>
+<wire x1="27.6225" y1="0" x2="27.6225" y2="27.305" width="0.1524" layer="20"/>
+<wire x1="27.6225" y1="27.305" x2="0" y2="27.305" width="0.1524" layer="20"/>
+<wire x1="0" y1="27.305" x2="0" y2="0" width="0.1524" layer="20"/>
 </plain>
 <attributes>
