File: hw/esp32_module.sch (EAGLE design)
At the start: 2 parts, among them IC1 ESP32-S2_WROVER, IC2 ESP32-WROVER

Commit message: improved
Parts:
- added BOOT, IO13, RESET: (no value), Ergaenzung:TASTER-9314_SMD
- added C1, C2: 0.1, rcl:C-EUC0805
- added C3, C4: 22p, rcl:C-EUC0805
- added C5: 10u, rcl:CPOL-EUB/3528-21W
- added C6: (no value), rcl:CPOL-EUC/6032-28R
- added D1: 4148, diode:DIODE-MINIMELF
- added GPS: GPS, con-amp-micromatch:MICROMATCH-6SMD
- added I2C, PROG: I2CBUS, con-amp-micromatch:MICROMATCH-10SMD
- added J_BO, J_BR, J_IO4, J_OLED1, J_OLED2, J_P1, J_P2, J_VCC: (no value), jumper:SJ2W
- added J_L1, J_L2, J_L3, J_L4, J_L5, J_L6, J_L7, J_L7B, J_L8, J_L8B, J_R6, J_R7, J_R8, J_RBO, J_RSO, J_U02R, J_U02T, J_VCCOUT: (no value), jumper:SJ
- added L, R: (no value), con-lstb:MA08-1
- added LED_B, LED_G: G, led:LEDCHIPLED_0805
- added LED_R: R, led:LEDCHIPLED_0805
- added OLED: (no value), con-lstb:MA04-1
- added Q2: IRLML2244, User-Submitted:MOSFET-PCHANNELIRLML2244
- added R1, R15, R19, R2, R25, R26, R27, R28, R29, R3, R30, R31, R32, R33, R34, R35, R36, R37, R38, R39, R4, R40, R41, R42, R5, R6, R7, R8, R9: (no value), rcl:R-EU_R0805
- added R10, R11, R12, R13, R14, R16, R17, R23, R43, R44, R45: 10k, rcl:R-EU_R0805
- added R18, R20, R21: (no value), rcl:R-EU_R0603
- added SDCARD: MICROSD_SD_MODE, con-molex-microsd:MICROSD_SD_MODE
- added SPI: SPIBUS, con-amp-micromatch:MICROMATCH-8SMD
- added T2: (no value), transistor:BC817-16-NPN-SOT23-BEC
Connections:
- new net BOOT: BOOT.2, IC1.IO0, IC2.IO0, J_BO.1, PROG-6.S, R11.1
- new net BUS_FON: I2C-3.S, IC1.IO16, IC2.SENSR_VN, R27.2
- new net BUS_INT: I2C-9.S, IC1.IO11, IC2.SENSR_VP, J_R8.2, R26.2
- new net BUS_ON: IC1.IO26, J_BO.2, J_BR.1, J_RBO.2, R23.1
- new net BUS_RESET: I2C-5.S, IC1.IO14, J_BR.2, J_IO4.3, J_L8.1, J_RBO.1, R28.2
- new net BUS_SCL: GPS-2.S, I2C-7.S, IC1.IO15, IC2.IO22, J_R7.2, R29.2
- new net BUS_SDA: GPS-4.S, I2C-1.S, IC1.IO13, IC2.IO21, J_R6.2, R25.2
- new net EN: C1.1, IC1.EN, IC2.EN, J_BO.3, PROG-5.S, R10.1, RESET.2
- new net LCD_1: J_OLED1.2, OLED.1
- new net LCD_2: J_OLED2.2, OLED.2
- new net MTCK: IC1.IO39, IC2.IO13, IO13.2, PROG-10.S, R1.2
- new net MTDI: IC1.IO41, IC2.IO12, PROG-7.S, R15.2, R20.2
- new net MTDO: IC1.IO40, IC2.IO15, PROG-9.S, R12.1, R2.2, R21.2
- new net MTMS: IC1.IO42, IC2.IO14, PROG-8.S, R3.2
- new net N$1: IC2.IO4, J_IO4.2
- new net N$12: J_R8.1, R.8
- new net N$18: R23.2, T2.B
- new net N$2: Q2.G, R45.2, T2.C
- new net N$20: LED_R.A, R20.1
- new net N$21: LED_B.A, R21.1
- new net N$24: J_L7.2, J_L7B.2, L.7
- new net N$25: J_L6.2, L.6, R19.1
- new net N$27: J_L8.2, J_L8B.2, L.8
- new net N$28: J_L5.2, L.5, R34.1
- new net N$29: J_L4.2, L.4, R35.1
- new net N$3: J_R6.1, R.6
- new net N$30: J_L2.2, L.2, R37.1
- new net N$31: J_L3.2, L.3, R36.1
- new net N$32: J_L1.2, L.1
- new net N$34: J_P2.2, PROG-2.S
- new net N$4: LED_G.A, R18.1
- new net N$5: J_R7.1, R.7
- new net N$6: J_P1.2, PROG-1.S
- new net OLED_SCL: IC1.IO12, IC2.IO27, J_L8B.1, OLED.3, R31.2
- new net OLED_SDA: IC1.IO10, IC2.IO26, J_L7B.1, OLED.4, R30.2
- new net S2_IO1: IC1.IO1, R37.2, R38.1
- new net S2_IO2: IC1.IO2, R36.2, R39.1
- new net S2_IO3: IC1.IO3, R35.2, R40.1
- new net S2_IO4: IC1.IO4, R34.2, R41.1
- new net S2_IO45: IC1.IO45, R16.1, R17.2
- new net S2_IO46: IC1.IO46, R43.1, R44.2
- new net S2_IO5: IC1.IO5, R19.2, R42.1
- new net SD_CLK: R3.1, R6.2, SDCARD.CLK
- new net SD_CMD: R2.1, R7.2, SDCARD.CMD
- new net SD_D0: IC1.IO21, IC2.IO2, R4.2, SDCARD.DATA0
- new net SD_D1: IC1.IO6, J_IO4.1, R5.2, SDCARD.DATA1
- new net SD_D2: R15.1, R9.2, SDCARD.DATA2
- new net SD_D3: R1.1, R8.2, SDCARD.CD/DATA3
- new net SPI_CS0: IC1.IO34, IC2.IO5, J_L5.1, R13.1, R14.2, SPI-7.S
- new net SPI_CS1: IC1.IO38, IC2.IO25, J_L6.1, SPI-8.S
- new net SPI_MISO: IC1.IO35, IC2.IO23, J_L2.1, SPI-1.S
- new net SPI_MOSI: IC1.IO37, IC2.IO19, J_L3.1, SPI-4.S
- new net SPI_ON: IC1.IO33, J_RSO.2
- new net SPI_RESET: IC1.IO8, J_BR.3, J_L7.1, J_RSO.1, SPI-5.S
- new net SPI_SCK: IC1.IO36, IC2.IO18, J_L4.1, SPI-3.S
- new net U0RXD: IC1.RXD0, IC2.RXD0, J_P1.3, J_U02R.1
- new net U0TXD: IC1.TXD0, IC2.TXD0, J_P2.3, J_U02T.1
- new net U1RXD: GPS-1.S, IC1.IO18, IC2.IO34
- new net U1TXD: GPS-3.S, IC1.IO17, IC2.IO32
- new net U2RXD: IC1.IO9, IC2.IO35, J_U02R.2, R33.2
- new net U2TXD: D1.C, IC1.IO7, IC2.IO33, J_U02T.2
- new net U2_BUS: D1.A, J_L1.1, R32.1, R33.1
- new net U33A: J_VCC.3, J_VCCOUT.2, R.2
- new net U33B: J_VCC.1, R.3
- new net U5: I2C-4.S, R.4
- new net UBAT: I2C-6.S, R.5
- new net UBUS: GPS-5.S, I2C-2.S, J_VCCOUT.1, Q2.D, SPI-2.S
- new net USBN: C4.1, IC1.IO19, J_P1.1
- new net USBP: C3.1, IC1.IO20, J_P2.1
- new net VCC: C2.1, C5.+, C6.+, IC1.3V3, IC2.3V3, J_OLED1.3, J_OLED2.3, J_VCC.2, PROG-3.S, Q2.S, R10.2, R11.2, R12.2, R13.2, R16.2, R18.2, R25.1, R26.1, R27.1, R28.1, R29.1, R30.1, R31.1, R32.2, R43.2, R45.1, R5.1, R6.1, R7.1, R8.1, R9.1, SDCARD.VDD
- net GND: now also BOOT.3, BOOT.4, C1.2, C2.2, C3.2, C4.2, C5.-, C6.-, GPS-6.S, I2C-10.S, I2C-8.S, IC1.GND4, IC2.GND2, IO13.3, IO13.4, J_OLED1.1, J_OLED2.1, LED_B.C, LED_G.C, LED_R.C, PROG-4.S, R.1, R14.1, R17.1, R38.2, R39.2, R4.1, R40.2, R41.2, R42.2, R44.1, RESET.3, RESET.4, SDCARD.VSS, SPI-6.S, T2.E
Other:
- note removed: "V1.0"
- moved on the sheet: IC1, IC2

Commit message: -
Parts:
- added R22: 10k, rcl:R-EU_R0805
Connections:
- net U1RXD: now also R22.1
- net VCC: now also R22.2
Changed lines of the file:
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@@
 <part name="P+12" library="supply1" library_urn="urn:adsk.eagle:library:371" deviceset="VCC" device=""/>
 <part name="P+13" library="supply1" library_urn="urn:adsk.eagle:library:371" deviceset="VCC" device=""/>
+<part name="R22" library="rcl" library_urn="urn:adsk.eagle:library:334" deviceset="R-EU_" device="R0805" package3d_urn="urn:adsk.eagle:package:23553/2" value="10k"/>
+<part name="P+26" library="supply1" library_urn="urn:adsk.eagle:library:371" deviceset="VCC" device=""/>
 </parts>
 <sheets>
@@
 <instance part="P+13" gate="VCC" x="58.42" y="114.3" smashed="yes" rot="R90">
 <attribute name="VALUE" x="60.96" y="111.76" size="1.778" layer="96" rot="R180"/>
+</instance>
+<instance part="R22" gate="G$1" x="22.86" y="63.5" smashed="yes" rot="MR180">
+<attribute name="NAME" x="19.05" y="62.0014" size="1.778" layer="95" rot="MR180"/>
+<attribute name="VALUE" x="19.05" y="66.802" size="1.778" layer="96" rot="MR180"/>
+</instance>
+<instance part="P+26" gate="VCC" x="30.48" y="63.5" smashed="yes" rot="R270">
+<attribute name="VALUE" x="27.94" y="66.04" size="1.778" layer="96"/>
 </instance>
 </instances>
@@
 <pinref part="P+13" gate="VCC" pin="VCC"/>
 </segment>
+<segment>
+<pinref part="R22" gate="G$1" pin="2"/>
+<pinref part="P+26" gate="VCC" pin="VCC"/>
+</segment>
 </net>
 <net name="N$20" class="0">
@@
 <wire x1="20.32" y1="58.42" x2="17.78" y2="58.42" width="0.1524" layer="91"/>
 <label x="20.32" y="58.42" size="1.778" layer="95" xref="yes"/>
-</segment>
-<segment>
+<pinref part="R22" gate="G$1" pin="1"/>
+<wire x1="17.78" y1="63.5" x2="17.78" y2="58.42" width="0.1524" layer="91"/>
+<junction x="17.78" y="58.42"/>
+</segment>
+<segment>
